File: usb-ic/usb-ic.kicad_sch (KiCad schematic)
At the start: 25 parts, among them SW1 SW_Push, U1 NE555P, U2 4017

Commit message: fixed schematic
Parts:
- removed R10, R11, R5, R6, R7, R8, R9: 330, Resistor_SMD:R_0805_2012Metric_Pad1.20x1.40mm_HandSolder, symbol Device:R
- R3: footprint Resistor_SMD:R_0805_2012Metric_Pad1.20x1.40mm_HandSolder -> (none)
- R4: value 330 -> 10k; footprint Resistor_SMD:R_0805_2012Metric_Pad1.20x1.40mm_HandSolder -> (none)
- SW1: footprint Button_Switch_SMD:SW_Push_SPST_NO_Alps_SKRK -> (none)
Connections:
- net at D2.2 (A): now also U2.2 (Q1); no longer R4.1
- net at R4.2: now also C1.2, R3.2, U1.1 (GND), U2.8 (VSS), U3.4 (GND); no longer U2.2 (Q1)
- net at D1.1 (K), D2.1 (K), D3.1 (K)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: now also R3.1; no longer C1.2, SW1.1, U1.1 (GND), U2.13 (CKEN), U2.8 (VSS), U3.4 (GND)
- net at U1.3 (Q), U2.14 (CLK): no longer SW1.2
- net at R1.1, U1.4 (R), U1.8 (VCC)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: now also SW1.1
- net at D1.2 (A): now also U2.3 (Q0); no longer R3.1
- net at D4.2 (A): now also U2.7 (Q3)
- net at D5.2 (A): now also U2.10 (Q4)
- net at D6.2 (A): now also U2.1 (Q5)
- net at D8.2 (A): now also U2.6 (Q7)
- net at D3.2 (A): now also U2.4 (Q2)
- net at D9.2 (A): now also U2.9 (Q8)
- net at D7.2 (A): now also U2.5 (Q6)
- new net: R4.1, SW1.2, U2.13 (CKEN)
